File: src/controller-pcb/hexalight.kicad_pcb (KiCad board)
At the start: 2 copper layers, 28 parts, among them J1 Conn_Coaxial_Power, J2 Conn_01x05, J3 Conn_01x03, J4 Conn_01x04, Q1 IRLB8721PBF, Q2 IRLB8721PBF, Q3 IRLB8721PBF, Q4 IRLB8721PBF, Q5 IRLB8721PBF, SW1 SW_Push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

Commit message: Updating CAD files
Parts:
- removed JP1: SolderJumper_3_Open, Connector_PinHeader_2.54mm:PinHeader_1x03_P2.54mm_Vertical
- removed Q1, Q2, Q3, Q4, Q5: IRLB8721PBF, Package_TO_SOT_THT:TO-220-3_Vertical
- removed TP1, TP10, TP2, TP3, TP4, TP5, TP6, TP7, TP8, TP9: TestPoint, TestPoint:TestPoint_Loop_D1.80mm_Drill1.0mm_Beaded
- added C4: 100nF, Capacitor_SMD:C_1210_3225Metric_Pad1.33x2.70mm_HandSolder, F.Cu at (142.3, 114.6)
- added C5: 100nF, Capacitor_SMD:C_0805_2012Metric_Pad1.18x1.45mm_HandSolder, F.Cu at (139.5, 102.5)
- added C6: 100nF, Capacitor_SMD:C_0805_2012Metric_Pad1.18x1.45mm_HandSolder, F.Cu at (142.5, 102.5)
- added C7: 22uF, Capacitor_SMD:C_0805_2012Metric_Pad1.18x1.45mm_HandSolder, F.Cu at (145.3, 102.5)
- added C8: 22uF, Capacitor_SMD:C_0805_2012Metric_Pad1.18x1.45mm_HandSolder, F.Cu at (148.2, 102.5)
- C1: footprint Capacitor_SMD:C_0603_1608Metric -> Capacitor_SMD:C_0805_2012Metric_Pad1.18x1.45mm_HandSolder
- C2: value 10uF -> 1uF; footprint Capacitor_SMD:C_1206_3216Metric -> Capacitor_SMD:C_0805_2012Metric_Pad1.18x1.45mm_HandSolder
- C3: value 100nF -> 22uF; footprint Capacitor_SMD:C_0603_1608Metric -> Capacitor_SMD:C_1210_3225Metric_Pad1.33x2.70mm_HandSolder
- J2: value Conn_01x05 -> Serial; footprint TerminalBlock_Phoenix:TerminalBlock_Phoenix_MPT-0,5-5-2.54_1x05_P2.54mm_Horizontal -> Connector_PinHeader_2.54mm:PinHeader_1x04_P2.54mm_Vertical
- J3: value Conn_01x03 -> Right Panel; footprint TerminalBlock_Phoenix:TerminalBlock_Phoenix_MPT-0,5-3-2.54_1x03_P2.54mm_Horizontal -> TE-Connectivity:119542892
- J4: value Conn_01x04 -> Left Panel; footprint Connector_JST:JST_XH_S4B-XH-A-1_1x04_P2.50mm_Horizontal -> TE-Connectivity:119542892
- R1: footprint Resistor_SMD:R_0603_1608Metric -> Resistor_SMD:R_0805_2012Metric_Pad1.20x1.40mm_HandSolder
- SW1: value SW_Push -> Reset; footprint Button_Switch_SMD:SW_Push_1P1T_NO_6x6mm_H9.5mm -> Button_Switch_SMD:SW_SPST_B3U-1000P
- SW2: value SW_Push -> Boot Option; footprint Button_Switch_SMD:SW_Push_1P1T_NO_6x6mm_H9.5mm -> Button_Switch_SMD:SW_SPST_B3U-1000P
- U2: value ESP32-WROOM-32 -> ESP32-WROOM-32E; footprint kicad-libraries:ESP32-WROOM-32 -> Espressif:ESP32-WROOM-32E
- moved J2 59.6 mm to (144.0, 67.3), turned to 90 degrees
- moved U2 54.8 mm to (148.3, 52.7)
- moved C2 48.7 mm to (146.3, 72.9), turned to 90 degrees
- moved R1 46.7 mm to (148.6, 72.9), turned to 90 degrees
- moved C1 41.7 mm to (143.8, 72.9), turned to 90 degrees
- moved J1 39.9 mm to (151.4, 114.7), turned to 90 degrees
- moved SW1 35.7 mm to (140.0, 70.4), turned to 90 degrees
- moved J3 23.5 mm to (157.6, 86.1)
- moved C3 18.5 mm to (142.3, 119.9), turned to 180 degrees
- moved J4 18.4 mm to (138.9, 86.1), turned to 180 degrees
- moved SW2 14.3 mm to (156.6, 70.4), turned to 90 degrees
- moved U1 13.1 mm to (153.7, 104.1), turned to 90 degrees
Connections:
- C1 pad 1: Net-(C1-Pad1) -> GND
- C1 pad 2: GND -> /RST
- C2 pad 2: +3V3 -> /RST
- C3 pad 1: GND -> +5V
- C3 pad 2: +3V3 -> GND
- J1 pad 1: B -> +5V
- J2 pad 1: B -> +3V3
- J2 pad 2: B -> /Rx
- J2 pad 3: B -> /Tx
- J2 pad 4: B -> GND
- J3 pad 1: B -> +5V
- J3 pad 2: DO -> LED_R
- J3 pad 3: GND -> TOUCH_R
- J4 pad 1: +3V3 -> +5V
- J4 pad 2: TX -> LED_L
- J4 pad 3: RX -> TOUCH_L
- R1 pad 2: Net-(C1-Pad1) -> /RST
- SW1 pad 1: Net-(C1-Pad1) -> GND
- SW1 pad 2: GND -> /RST
- SW2 pad 1: TOUCH_0 -> GND
- SW2 pad 2: GND -> Net-(SW2-Pad2)
- U1 pad 3: B -> +5V
- U2 pad 10: Net-(U2-Pad10) -> unconnected-(U2-Pad10)
- U2 pad 11: Net-(U2-Pad11) -> unconnected-(U2-Pad11)
- U2 pad 12: Net-(U2-Pad12) -> unconnected-(U2-Pad12)
- U2 pad 13: Net-(U2-Pad13) -> unconnected-(U2-Pad13)
- U2 pad 14: Net-(U2-Pad14) -> unconnected-(U2-Pad14)
- U2 pad 16: Net-(U2-Pad16) -> unconnected-(U2-Pad16)
- U2 pad 17: Net-(U2-Pad17) -> unconnected-(U2-Pad17)
- U2 pad 18: Net-(U2-Pad18) -> unconnected-(U2-Pad18)
- U2 pad 19: Net-(U2-Pad19) -> unconnected-(U2-Pad19)
- U2 pad 20: Net-(U2-Pad20) -> unconnected-(U2-Pad20)
- U2 pad 21: Net-(U2-Pad21) -> unconnected-(U2-Pad21)
- U2 pad 22: Net-(U2-Pad22) -> unconnected-(U2-Pad22)
- U2 pad 23: Net-(U2-Pad23) -> unconnected-(U2-Pad23)
- U2 pad 24: Net-(U2-Pad24) -> unconnected-(U2-Pad24)
- U2 pad 25: TOUCH_0 -> Net-(SW2-Pad2)
- U2 pad 26: TOUCH_1 -> unconnected-(U2-Pad26)
- U2 pad 27: SDO -> unconnected-(U2-Pad27)
- U2 pad 28: SCK -> unconnected-(U2-Pad28)
- U2 pad 29: Net-(U2-Pad29) -> unconnected-(U2-Pad29)
- U2 pad 3: Net-(C1-Pad1) -> /RST
- U2 pad 30: LED_DO -> unconnected-(U2-Pad30)
- U2 pad 31: LED_W -> unconnected-(U2-Pad31)
- U2 pad 32: Net-(U2-Pad32) -> unconnected-(U2-Pad32)
- U2 pad 33: LED_B -> unconnected-(U2-Pad33)
- U2 pad 34: RX -> /Rx
- U2 pad 35: TX -> /Tx
- U2 pad 36: LED_G -> LED_R
- U2 pad 37: LED_R -> LED_L
- U2 pad 39: GND -> (no net)
- U2 pad 4: Net-(U2-Pad4) -> unconnected-(U2-Pad4)
- U2 pad 5: Net-(U2-Pad5) -> unconnected-(U2-Pad5)
- U2 pad 6: Net-(U2-Pad6) -> unconnected-(U2-Pad6)
- U2 pad 7: Net-(U2-Pad7) -> unconnected-(U2-Pad7)
- U2 pad 8: Net-(U2-Pad8) -> TOUCH_L
- U2 pad 9: Net-(U2-Pad9) -> TOUCH_R
Routing:
- net GND: track 0.00 -> 91.7 mm, vias 0 -> 9
- net +3V3: track 0.00 -> 91.4 mm, vias 0 -> 3
- net +5V: track 0.00 -> 72.1 mm, vias 0 -> 2
- net LED_L: track 0.00 -> 59.4 mm, vias 0 -> 2
- net TOUCH_R: track 0.00 -> 45.5 mm, vias 0 -> 2
- net LED_R: track 0.00 -> 43.6 mm, vias 0 -> 2
- net TOUCH_L: track 0.00 -> 36.7 mm, vias 0 -> 2
- net /RST: track 0.00 -> 33.4 mm
- net /Tx: track 0.00 -> 25.4 mm, vias 0 -> 1
- net /Rx: track 0.00 -> 25.3 mm, vias 0 -> 1
- net (no net): track 0.00 -> 17.2 mm
- net Net-(SW2-Pad2): track 0.00 -> 6.60 mm
- added copper zone on B.Cu, net GND
Other:
- board outline added: 21 x 81.2 mm
- net class Default removed
- board text added: "+5V"
- board text added: "3V3"
- board text added: "Boot Sel"
- board text added: "GND"
- board text added: "Hexalight"
- board text added: "JLCJLCJLCJLC"
- board text added: "Rst"
- board text added: "Rx"
- board text added: "Tx"
